Commit message: Added all code to control arm via sensors. Also contact detection.

File: jaco_arm/jaco_description/urdf/jaco.urdf.xacro (robot description, xacro)
@@ -757,5 +757,5 @@
       </material>
     </visual>
-    <collision>
+    <collision name = "index_collision">
       <origin xyz="0 0 0" rpy="${M_PI} ${M_PI_4+M_PI_4/2.0} 0" />
       <geometry>
@@ -764,4 +764,13 @@
     </collision>
   </link>
+  <gazebo reference="${jaco_prefix}_8_finger_index">
+    <sensor name='index_contact' type='contact'>
+    	<plugin name="my_plugin" filename="libindex_contact.so"/>
+        <contact>
+        	<collision>${jaco_prefix}_8_finger_index_collision</collision>
+        </contact>
+        <update_rate> 5 </update_rate>
+    </sensor>
+  </gazebo>
     <joint name="${jaco_prefix}_finger_joint_0" type="revolute">
      <xacro:damping_fingers/>
@@ -845,5 +854,5 @@
       </material>
     </visual>
-    <collision>
+    <collision name = "thumb_collision">
       <origin xyz="0 0 0" rpy="${M_PI} ${M_PI_4+M_PI_4/2.0} 0" />
       <geometry>
@@ -852,4 +861,13 @@
     </collision>
   </link>
+    <gazebo reference="${jaco_prefix}_8_finger_thumb">
+    <sensor name='thumb_contact' type='contact'>
+    	<plugin name="thumb_plugin" filename="thumb_contact.so"/>
+        <contact>
+        	<collision>${jaco_prefix}_8_finger_thumb_collision</collision>
+        </contact>
+        <update_rate> 5 </update_rate>
+    </sensor>
+  </gazebo>
     <joint name="${jaco_prefix}_finger_joint_2" type="revolute">
      <xacro:damping_fingers/>

Commit message: Did a lot of stuff. All 3 fingers working with contact sensors. Also uploading Arduino file

File: jaco_arm/jaco_description/urdf/jaco.urdf.xacro (robot description, xacro)
@@ -681,5 +681,5 @@
     </visual>
      <xacro:testSphere/>
-    <collision>
+    <collision name = "limb_collision">
       <origin xyz="0 0 0" rpy="0 0 0" />
       <geometry>
@@ -711,5 +711,5 @@
   </joint>
   <!-- ...........................  -->
-  <!--      FINGERS          -->
+  <!--             FINGERS          -->
   <!-- ...........................  -->
   <link name="${jaco_prefix}_7_finger_mount_index">
@@ -863,5 +863,5 @@
     <gazebo reference="${jaco_prefix}_8_finger_thumb">
     <sensor name='thumb_contact' type='contact'>
-    	<plugin name="thumb_plugin" filename="thumb_contact.so"/>
+    	<plugin name="thumb_plugin" filename="libthumb_contact.so"/>
         <contact>
         	<collision>${jaco_prefix}_8_finger_thumb_collision</collision>
@@ -950,5 +950,5 @@
       </material>
     </visual>
-    <collision>
+    <collision name = "pinkie_collision">
       <origin xyz="0 0 0" rpy="${M_PI} ${M_PI_4+M_PI_4/2.0} 0" />
       <geometry>
@@ -957,4 +957,13 @@
     </collision>
   </link>
+  <gazebo reference="${jaco_prefix}_8_finger_pinkie">
+    <sensor name='pinkie_contact' type='contact'>
+      <plugin name="pinkie_plugin" filename="libmiddle_contact.so"/>
+        <contact>
+          <collision>${jaco_prefix}_8_finger_pinkie_collision</collision>
+        </contact>
+        <update_rate> 5 </update_rate>
+    </sensor>
+  </gazebo>
     <joint name="${jaco_prefix}_finger_joint_4" type="revolute">
     <xacro:damping_fingers/>

Commit message: fixed the build to work in ROS Melodic

File: jaco_arm/jaco_description/urdf/jaco.urdf.xacro (robot description, xacro)
@@ -681,5 +681,5 @@
     </visual>
      <xacro:testSphere/>
-    <collision name = "limb_collision">
+    <collision>
       <origin xyz="0 0 0" rpy="0 0 0" />
       <geometry>
@@ -711,5 +711,5 @@
   </joint>
   <!-- ...........................  -->
-  <!--             FINGERS          -->
+  <!--      FINGERS          -->
   <!-- ...........................  -->
   <link name="${jaco_prefix}_7_finger_mount_index">
@@ -757,5 +757,5 @@
       </material>
     </visual>
-    <collision name = "index_collision">
+    <collision>
       <origin xyz="0 0 0" rpy="${M_PI} ${M_PI_4+M_PI_4/2.0} 0" />
       <geometry>
@@ -766,9 +766,9 @@
   <gazebo reference="${jaco_prefix}_8_finger_index">
     <sensor name='index_contact' type='contact'>
-    	<plugin name="my_plugin" filename="libindex_contact.so"/>
+      <plugin name="my_plugin" filename="libindex_contact.so" />
         <contact>
-        	<collision>${jaco_prefix}_8_finger_index_collision</collision>
+          <collision>${jaco_prefix}_8_finger_index_collision</collision>
         </contact>
-        <update_rate> 5 </update_rate>
+        <update_rate> 50 </update_rate>
     </sensor>
   </gazebo>
@@ -854,5 +854,5 @@
       </material>
     </visual>
-    <collision name = "thumb_collision">
+    <collision>
       <origin xyz="0 0 0" rpy="${M_PI} ${M_PI_4+M_PI_4/2.0} 0" />
       <geometry>
@@ -861,11 +861,11 @@
     </collision>
   </link>
-    <gazebo reference="${jaco_prefix}_8_finger_thumb">
+  <gazebo reference="${jaco_prefix}_8_finger_thumb">
     <sensor name='thumb_contact' type='contact'>
-    	<plugin name="thumb_plugin" filename="libthumb_contact.so"/>
+      <plugin name="thumb_plugin" filename="libthumb_contact.so"/>
         <contact>
-        	<collision>${jaco_prefix}_8_finger_thumb_collision</collision>
+          <collision>${jaco_prefix}_8_finger_thumb_collision</collision>
         </contact>
-        <update_rate> 5 </update_rate>
+        <update_rate> 50 </update_rate>
     </sensor>
   </gazebo>
@@ -950,5 +950,5 @@
       </material>
     </visual>
-    <collision name = "pinkie_collision">
+    <collision>
       <origin xyz="0 0 0" rpy="${M_PI} ${M_PI_4+M_PI_4/2.0} 0" />
       <geometry>
@@ -963,5 +963,5 @@
           <collision>${jaco_prefix}_8_finger_pinkie_collision</collision>
         </contact>
-        <update_rate> 5 </update_rate>
+        <update_rate> 50 </update_rate>
     </sensor>
   </gazebo>

File: jaco_tutorial/jaco_on_table/urdf/jaco_on_table.urdf.xacro (robot description, xacro)
@@ -14,31 +14,31 @@
   <xacro:arg name="add_transmission_pos" default="false"/>
   <xacro:arg name="add_transmission_vel" default="false"/>
-	<joint name="base_to_jaco_on_table" type="fixed">
-		<xacro:insert_block name="origin" />
-		<parent link="${parent}" />
-		<child link="robot_base" />
-	</joint>
-	<link name="robot_base">
-		<static>false</static>
-	</link>
-	<xacro:include filename="$(find jaco_on_table)/urdf/objects/table.xacro" />
-	<joint name="table_to_arm" type="fixed">
-		<origin xyz="0.40488474042 0.27988474042 0.3" rpy="0 0 -0.785398163397458" />
-		<parent link="robot_base"/>
-		<child link="table_base"/>
-	</joint>
+  <joint name="base_to_jaco_on_table" type="fixed">
+    <xacro:insert_block name="origin" />
+    <parent link="${parent}" />
+    <child link="robot_base" />
+  </joint>
+  <link name="robot_base">
+    <static>false</static>
+  </link>
+  <xacro:include filename="$(find jaco_on_table)/urdf/objects/table.xacro" />
+  <joint name="table_to_arm" type="fixed">
+    <origin xyz="0.40488474042 0.27988474042 0.3" rpy="0 0 -0.785398163397458" />
+    <parent link="robot_base"/>
+    <child link="table_base"/>
+  </joint>
   <xacro:arm_stand_link link_name="arm_stand"/>
-	<joint name="j2b" type="fixed">
-		<origin xyz="0 -0.035 0" rpy="-1.57079632679 -3.14159265358979 0" /> <!-- set the arm "inside" the table for now because of the rim along the real table. creating a bit of a buffer zone so moveit trajectories are within safe distance of the table edges. -->
-		<parent link="tabletop_corner" />
-		<child link="arm_stand" />
-		<axis xyz="0 0 0" />
-	</joint>
-	<!-- Add the JACO arm to the given parent link with the given transforms -->
+  <joint name="j2b" type="fixed">
+    <origin xyz="0 -0.035 0" rpy="-1.57079632679 -3.14159265358979 0" /> <!-- set the arm "inside" the table for now because of the rim along the real table. creating a bit of a buffer zone so moveit trajectories are within safe distance of the table edges. -->
+    <parent link="tabletop_corner" />
+    <child link="arm_stand" />
+    <axis xyz="0 0 0" />
+  </joint>
+  <!-- Add the JACO arm to the given parent link with the given transforms -->
   <xacro:jaco_arm parent="arm_stand" mass_divider="2" finger_mass_divider="1">
     <origin xyz="-0.000482247085224208 0.08 -0.000503436190578577" rpy="1.57079632679 0 3.14159265359" />
     <xacro:arg name="add_transmission_pos" default="$(arg add_transmission_pos)"/>
     <xacro:arg name="add_transmission_vel" default="$(arg add_transmission_vel)"/>
-	</xacro:jaco_arm>
+  </xacro:jaco_arm>
   <!-- Optional: Add the Xtion to the table to observe the real arm -->
   <xacro:if value="$(arg sensor_on_table)">
